Commit message: Update robotarm_description.urdf

File: URDF_model/bmirobot_description/urdf/robotarm_description.urdf (robot description, URDF)
Before this commit: robot robotarm, 25 links, 24 joints
Links:
- link right_hand1: geometry collision mesh filename=package://bmirobot_description/modle/stl_V5/hand-1.dae; visual mesh filename=package://bmirobot_description/modle/stl_V5/hand-1.dae
- link right_hand2: geometry collision mesh filename=package://bmirobot_description/modle/stl_V5/hand-2.dae; visual mesh filename=package://bmirobot_description/modle/stl_V5/hand-2.dae

Commit message: multiprocess version

File: URDF_model/bmirobot_description/urdf/robotarm_description.urdf (robot description, URDF)
Before this commit: robot robotarm, 25 links, 24 joints
Links:
- link left_hand1: geometry collision mesh filename=package://bmirobot_description/modle/stl_V5/left-hand-1.dae; visual mesh filename=package://bmirobot_description/modle/stl_V5/left-hand-1.dae
- link left_hand2: geometry collision mesh filename=package://bmirobot_description/modle/stl_V5/left-hand-2.dae; visual mesh filename=package://bmirobot_description/modle/stl_V5/left-hand-2.dae
- link left_link8: geometry collision mesh filename=package://bmirobot_description/modle/stl_V5/left-link7.dae; visual mesh filename=package://bmirobot_description/modle/stl_V5/left-link7.dae
Joints:
- joint left_hand_joint1: axis 0 0 1 -> 0 1 0
- joint left_hand_joint2: axis 0 0 1 -> 0 1 0; limit lower=-0.785398163397 upper=0.0 effort=1000.0 velocity=9.42477796077 -> lower=-1.74532925199 upper=1.74532925199 effort=1000.0 velocity=9.42477796077; origin xyz=0.0865 0 0.024 rpy=0 0 0 -> xyz=0.0865 0.024 0 rpy=0 0 0
- joint left_joint7: origin xyz=0.0 0 0 rpy=0.0 0 0 -> xyz=0.0 0 0 rpy=1.57079632679 0 0

File: URDF_model/cube_small_pick.urdf (robot description, URDF)
Before this commit: robot cube.urdf, 1 links, 0 joints
Links:
- link baseLink: mass 2 -> 1; geometry collision box size=.06 .06 .06; visual box size=.06 .06 .06

File: URDF_model/cube_small_push.urdf (robot description, URDF)
Before this commit: robot cube.urdf, 1 links, 0 joints
Links:
- link baseLink: geometry collision box size=.06 .06 .06; visual box size=.06 .06 .06

File: URDF_model/cube_small_target_pick.urdf (robot description, URDF)
Before this commit: robot cube.urdf, 1 links, 0 joints
Links:
- link baseLink: geometry visual box size=.06 .06 .06

File: URDF_model/cube_small_target_push.urdf (robot description, URDF)
Before this commit: robot cube.urdf, 1 links, 0 joints
Links:
- link baseLink: geometry visual box size=.05 .05 .05
